File: hardware/mixsid.sch (KiCad schematic (older format))
At the start: 76 parts, among them P1 INPUT, P2 CONTROL, P3 RAW, P4 SOCKET LEFT, P5 OUTPUT, P6 SOCKET RIGHT, Q1 BC547, Q2 BC547, U1 GAL16V8, U2 SID2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

Commit message: MixSID_SMD
Parts:
- C1, C10, C11, C12, C13, C14, C2, C23, C24, C25, C26, C27, C3, C4, C5, C6, C7, C8, C9: footprint Pinheaders:C_Disc_D3_P2.5 -> Pinheaders:0805; symbol C_Small -> mixsid-rescue:C_Small-1
- C15, C16, C20, C21: footprint Pinheaders:C_Disc_D3_P2.5 -> Pinheaders:0805; symbol C -> mixsid-rescue:C-1
- C17, C18: footprint Pinheaders:C_Radial_D5_L6_P2.5 -> Pinheaders:0805; symbol CP1_Small -> mixsid-rescue:CP1_Small-1
- C19, C22: footprint Pinheaders:C_Radial_D5_L6_P2.5 -> Pinheaders:0805; symbol CP_Small -> mixsid-rescue:CP_Small-1
- D1, D2: value 1N4002 -> S1A; footprint Discret:DO-41 -> Pinheaders:DO-214AC; symbol D -> mixsid-rescue:D-1
- JP1, JP11, JP12, JP13, JP2, JP3, JP4, JP5, JP6, JP7, JP8: symbol JUMPER3 -> mixsid-rescue:JUMPER3-1
- JP10, JP9: symbol JUMPER -> mixsid-rescue:JUMPER-1
- P1: value INPUT -> INPUT DF13-5P; footprint Pinheaders:Pin_Header_Straight_1x05 -> Pinheaders:DF13-5P; symbol CONN_01X05 -> mixsid-rescue:CONN_01X05-1
- P2: symbol CONN_02X06 -> mixsid-rescue:CONN_02X06-1
- P3: symbol CONN_01X02 -> mixsid-rescue:CONN_01X02-1
- P4, P6: symbol CONN_01X14 -> mixsid-rescue:CONN_01X14-1
- P5: value OUTPUT -> OUTPUT DF13-3P; footprint Pinheaders:Pin_Header_Straight_1x03 -> Pinheaders:DF13-3P; symbol CONN_01X03 -> mixsid-rescue:CONN_01X03-1
- Q1, Q2: value BC547 -> BCP54; footprint TO_SOT_Packages_THT:TO-92_Inline_Narrow_Oval -> Package_TO_SOT_SMD:SOT-223; symbol Q_NPN_CBE -> Transistor_BJT:BCP51
- R1, R10, R11, R12, R13, R14, R4, R5, R6, R7, R8: footprint Discret:R1 -> Pinheaders:0805; symbol R -> mixsid-rescue:R-1
- R2, R9: footprint Discret:R1 -> Pinheaders:0805; symbol R_Small -> mixsid-rescue:R_Small-1
- RV1, RV2, RV3, RV4: symbol POT -> mixsid-rescue:POT-1
- U1: symbol MIXSID -> mixsid-rescue:MIXSID-1
- U2, U5: symbol MOS6581 -> mixsid-rescue:MOS6581-1
- U3: footprint Pinheaders:TO-220 -> Package_TO_SOT_SMD:TO-252-2; symbol 7805 -> mixsid-rescue:1_7805-1
- U4: footprint Pinheaders:TO-220 -> Package_TO_SOT_SMD:TO-252-2; symbol 7805 -> mixsid-rescue:7805-1
- U6: footprint Pinheaders:DIP-16_W7.62mm -> Pinheaders:SOIC-16; symbol 4052 -> mixsid-rescue:4052-1
- U7: footprint Pinheaders:DIP-16_W7.62mm -> Pinheaders:SOIC-16; symbol 4053 -> mixsid-rescue:4053-1
- U8: footprint Pinheaders:DIP-8_W7.62mm -> Pinheaders:SOIC-8; symbol ICL7660 -> mixsid-rescue:ICL7660-1
- e1: renamed from R3; footprint Discret:R1 -> Pinheaders:0805; symbol R -> mixsid-rescue:R-1
Connections:
- net labels added: 1_VDD, GND-1
- wire segments 94 -> 122
